Commit message: Flatten Dex5 models into host URDF
Co-authored-by: Mertsr <115826687+Mertsr@users.noreply.github.com>

File: workspace/src/g1_description/urdf/g1_29dof_with_hand_rev_1_0.urdf (robot description, URDF)
Before this commit: robot g1_29dof_with_hand_rev_1_0, 37 links, 36 joints
Links:
- added link left_dex5_base_link, mass 0.090; collision mesh filename=package://g1_description/meshes/dex5_left/base_link.STL; visual mesh filename=package://g1_description/meshes/dex5_left/base_link.STL
- added link left_hand_grasp_frame
- added link left_index_1, mass 0.018690000000000002; collision mesh filename=package://g1_description/meshes/dex5_left/left_index_1.STL; visual mesh filename=package://g1_description/meshes/dex5_left/left_index_1.STL
- added link left_index_2, mass 0.01102; collision mesh filename=package://g1_description/meshes/dex5_left/left_index_2.STL; visual mesh filename=package://g1_description/meshes/dex5_left/left_index_2.STL
- added link left_index_force_sensor_1, mass 0.00020279; collision mesh filename=package://g1_description/meshes/dex5_left/left_index_force_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; visual mesh filename=package://g1_description/meshes/dex5_left/left_index_force_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
- added link left_index_force_sensor_2, mass 0.000255748193489171; collision mesh filename=package://g1_description/meshes/dex5_left/left_index_force_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; visual mesh filename=package://g1_description/meshes/dex5_left/left_index_force_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
- added link left_index_force_sensor_3, mass 6.79653902597574E-05; collision mesh filename=package://g1_description/meshes/dex5_left/left_index_force_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; visual mesh filename=package://g1_description/meshes/dex5_left/left_index_force_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
- added link left_little_1, mass 0.018690000000000002; collision mesh filename=package://g1_description/meshes/dex5_left/left_little_1.STL; visual mesh filename=package://g1_description/meshes/dex5_left/left_little_1.STL
- added link left_little_2, mass 0.018690000000000002; collision mesh filename=package://g1_description/meshes/dex5_left/left_little_2.STL; visual mesh filename=package://g1_description/meshes/dex5_left/left_little_2.STL
- added link left_little_force_sensor_1, mass 0.000202794502264302; collision mesh filename=package://g1_description/meshes/dex5_left/left_little_force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; visual mesh filename=package://g1_description/meshes/dex5_left/left_little_force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
- added link left_little_force_sensor_2, mass 0.00028024674848609; collision mesh filename=package://g1_description/meshes/dex5_left/left_little_force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; visual mesh filename=package://g1_description/meshes/dex5_left/left_little_force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
- added link left_little_force_sensor_3, mass 6.1053667014177E-05; collision mesh filename=package://g1_description/meshes/dex5_left/left_little_force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; visual mesh filename=package://g1_description/meshes/dex5_left/left_little_force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
- added link left_middle_1, mass 0.01866; collision mesh filename=package://g1_description/meshes/dex5_left/left_middle_1.STL; visual mesh filename=package://g1_description/meshes/dex5_left/left_middle_1.STL
- added link left_middle_2, mass 0.01767; collision mesh filename=package://g1_description/meshes/dex5_left/left_middle_2.STL; visual mesh filename=package://g1_description/meshes/dex5_left/left_middle_2.STL
- added link left_middle_force_sensor_1, mass 0.000202794522112893; collision mesh filename=package://g1_description/meshes/dex5_left/left_middle_force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; visual mesh filename=package://g1_description/meshes/dex5_left/left_middle_force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
- added link left_middle_force_sensor_2, mass 0.000262573593923136; collision mesh filename=package://g1_description/meshes/dex5_left/left_middle_force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; visual mesh filename=package://g1_description/meshes/dex5_left/left_middle_force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
- added link left_middle_force_sensor_3, mass 6.64914272946078E-05; collision mesh filename=package://g1_description/meshes/dex5_left/left_middle_force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; visual mesh filename=package://g1_description/meshes/dex5_left/left_middle_force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
- added link left_plam_1, mass 0.38382; collision mesh filename=package://g1_description/meshes/dex5_left/left_plam_1.STL; visual mesh filename=package://g1_description/meshes/dex5_left/left_plam_1.STL
- added link left_plam_2, mass 0.0205046589058927; collision mesh filename=package://g1_description/meshes/dex5_left/left_plam_2.STL; visual mesh filename=package://g1_description/meshes/dex5_left/left_plam_2.STL
- added link left_plam_force_sensor, mass 0.00240886556268154; collision mesh filename=package://g1_description/meshes/dex5_left/left_plam_force_s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; visual mesh filename=package://g1_description/meshes/dex5_left/left_plam_force_s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
- added link left_ring_1, mass 0.018690000000000002; collision mesh filename=package://g1_description/meshes/dex5_left/left_ring_1.STL; visual mesh filename=package://g1_description/meshes/dex5_left/left_ring_1.STL
- added link left_ring_2, mass 0.01102; collision mesh filename=package://g1_description/meshes/dex5_left/left_ring_2.STL; visual mesh filename=package://g1_description/meshes/dex5_left/left_ring_2.STL
- added link left_ring_force_sensor_1, mass 0.000202794434376476; collision mesh filename=package://g1_description/meshes/dex5_left/left_ring_force_s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; visual mesh filename=package://g1_description/meshes/dex5_left/left_ring_force_s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
- added link left_ring_force_sensor_2, mass 0.000255748190883527; collision mesh filename=package://g1_description/meshes/dex5_left/left_ring_force_s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; visual mesh filename=package://g1_description/meshes/dex5_left/left_ring_force_s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
- added link left_ring_force_sensor_3, mass 6.79657634628817E-05; collision mesh filename=package://g1_description/meshes/dex5_left/left_ring_force_s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; visual mesh filename=package://g1_description/meshes/dex5_left/left_ring_force_s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
- added link left_thumb_1, mass 0.01537; collision mesh filename=package://g1_description/meshes/dex5_left/left_thumb_1.STL; visual mesh filename=package://g1_description/meshes/dex5_left/left_thumb_1.STL
- added link left_thumb_2, mass 0.11034000000000001; collision mesh filename=package://g1_description/meshes/dex5_left/left_thumb_2.STL; visual mesh filename=package://g1_description/meshes/dex5_left/left_thumb_2.STL
- added link left_thumb_3, mass 0.01779; collision mesh filename=package://g1_description/meshes/dex5_left/left_thumb_3.STL; visual mesh filename=package://g1_description/meshes/dex5_left/left_thumb_3.STL
- added link left_thumb_4, mass 0.00766; collision mesh filename=package://g1_description/meshes/dex5_left/left_thumb_4.STL; visual mesh filename=package://g1_description/meshes/dex5_left/left_thumb_4.STL
- added link left_thumb_force_sensor_1, mass 0.000234351522411044; collision mesh filename=package://g1_description/meshes/dex5_left/left_thumb_force_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; visual mesh filename=package://g1_description/meshes/dex5_left/left_thumb_force_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
- added link left_thumb_force_sensor_2, mass 0.000119024235960817; collision mesh filename=package://g1_description/meshes/dex5_left/left_thumb_force_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; visual mesh filename=package://g1_description/meshes/dex5_left/left_thumb_force_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
- added link left_thumb_force_sensor_3, mass 0.000169894176021865; collision mesh filename=package://g1_description/meshes/dex5_left/left_thumb_force_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; visual mesh filename=package://g1_description/meshes/dex5_left/left_thumb_force_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
- added link left_thumb_force_sensor_4, mass 1.66991074236564E-05; collision mesh filename=package://g1_description/meshes/dex5_left/left_thumb_force_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; visual mesh filename=package://g1_description/meshes/dex5_left/left_thumb_force_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
- added link right_dex5_base_link, mass 0.090; collision mesh filename=package://g1_description/meshes/dex5_right/base_link.STL; visual mesh filename=package://g1_description/meshes/dex5_right/base_link.STL
- added link right_hand_grasp_frame
- added link right_index_1, mass 0.018690000000000002; collision mesh filename=package://g1_description/meshes/dex5_right/right_index_1.STL; visual mesh filename=package://g1_description/meshes/dex5_right/right_index_1.STL
- added link right_index_2, mass 0.01102; collision mesh filename=package://g1_description/meshes/dex5_right/right_index_2.STL; visual mesh filename=package://g1_description/meshes/dex5_right/right_index_2.STL
- added link right_index_force_sensor_1, mass 0.00020277926206694; collision mesh filename=package://g1_description/meshes/dex5_right/right_index_forc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; visual mesh filename=package://g1_description/meshes/dex5_right/right_index_forc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
- added link right_index_force_sensor_2, mass 0.000255748458180208; collision mesh filename=package://g1_description/meshes/dex5_right/right_index_forc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; visual mesh filename=package://g1_description/meshes/dex5_right/right_index_forc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
- added link right_index_force_sensor_3, mass 6.79646984897729E-05; collision mesh filename=package://g1_description/meshes/dex5_right/right_index_forc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; visual mesh filename=package://g1_description/meshes/dex5_right/right_index_forc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
- added link right_little_1, mass 0.018690000000000002; collision mesh filename=package://g1_description/meshes/dex5_right/right_little_1.S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; visual mesh filename=package://g1_description/meshes/dex5_right/right_little_1.S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
- added link right_little_2, mass 0.01166; collision mesh filename=package://g1_description/meshes/dex5_right/right_little_2.S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; visual mesh filename=package://g1_description/meshes/dex5_right/right_little_2.S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
- added link right_little_force_sensor_1, mass 0.000202779290224811; collision mesh filename=package://g1_description/meshes/dex5_right/right_little_for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; visual mesh filename=package://g1_description/meshes/dex5_right/right_little_for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
- added link right_little_force_sensor_2, mass 0.000280265363825451; collision mesh filename=package://g1_description/meshes/dex5_right/right_little_for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; visual mesh filename=package://g1_description/meshes/dex5_right/right_little_for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
- added link right_little_force_sensor_3, mass 6.10539921684107E-05; collision mesh filename=package://g1_description/meshes/dex5_right/right_little_for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; visual mesh filename=package://g1_description/meshes/dex5_right/right_little_for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
- added link right_middle_1, mass 0.01866; collision mesh filename=package://g1_description/meshes/dex5_right/right_middle_1.S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; visual mesh filename=package://g1_description/meshes/dex5_right/right_middle_1.S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
- added link right_middle_2, mass 0.01767; collision mesh filename=package://g1_description/meshes/dex5_right/right_middle_2.S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; visual mesh filename=package://g1_description/meshes/dex5_right/right_middle_2.S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
- added link right_middle_force_sensor_1, mass 0.000202779388301744; collision mesh filename=package://g1_description/meshes/dex5_right/right_middle_for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; visual mesh filename=package://g1_description/meshes/dex5_right/right_middle_for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
- added link right_middle_force_sensor_2, mass 0.00026259331441686; collision mesh filename=package://g1_description/meshes/dex5_right/right_middle_for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; visual mesh filename=package://g1_description/meshes/dex5_right/right_middle_for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
- added link right_middle_force_sensor_3, mass 6.64914575467581E-05; collision mesh filename=package://g1_description/meshes/dex5_right/right_middle_for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; visual mesh filename=package://g1_description/meshes/dex5_right/right_middle_for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
- added link right_plam_1, mass 0.38382; collision mesh filename=package://g1_description/meshes/dex5_right/right_plam_1.STL; visual mesh filename=package://g1_description/meshes/dex5_right/right_plam_1.STL
- added link right_plam_2, mass 0.0205048839537772; collision mesh filename=package://g1_description/meshes/dex5_right/right_plam_2.STL; visual mesh filename=package://g1_description/meshes/dex5_right/right_plam_2.STL
- added link right_plam_force_sensor, mass 0.00240887838334331; collision mesh filename=package://g1_description/meshes/dex5_right/right_plam_force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; visual mesh filename=package://g1_description/meshes/dex5_right/right_plam_force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
- added link right_ring_1, mass 0.018690000000000002; collision mesh filename=package://g1_description/meshes/dex5_right/right_ring_1.STL; visual mesh filename=package://g1_description/meshes/dex5_right/right_ring_1.STL
- added link right_ring_2, mass 0.01102; collision mesh filename=package://g1_description/meshes/dex5_right/right_ring_2.STL; visual mesh filename=package://g1_description/meshes/dex5_right/right_ring_2.STL
- added link right_ring_force_sensor_1, mass 0.00020277922338036; collision mesh filename=package://g1_description/meshes/dex5_right/right_ring_force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; visual mesh filename=package://g1_description/meshes/dex5_right/right_ring_force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
- added link right_ring_force_sensor_2, mass 0.00025574845564278; collision mesh filename=package://g1_description/meshes/dex5_right/right_ring_force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; visual mesh filename=package://g1_description/meshes/dex5_right/right_ring_force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
- added link right_ring_force_sensor_3, mass 6.79650392240318E-05; collision mesh filename=package://g1_description/meshes/dex5_right/right_ring_force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; visual mesh filename=package://g1_description/meshes/dex5_right/right_ring_force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
- added link right_thumb_1, mass 0.01537; collision mesh filename=package://g1_description/meshes/dex5_right/right_thumb_1.STL; visual mesh filename=package://g1_description/meshes/dex5_right/right_thumb_1.STL
- added link right_thumb_2, mass 0.11034000000000001; collision mesh filename=package://g1_description/meshes/dex5_right/right_thumb_2.STL; visual mesh filename=package://g1_description/meshes/dex5_right/right_thumb_2.STL
- added link right_thumb_3, mass 0.01779; collision mesh filename=package://g1_description/meshes/dex5_right/right_thumb_3.STL; visual mesh filename=package://g1_description/meshes/dex5_right/right_thumb_3.STL
- added link right_thumb_4, mass 0.00766; collision mesh filename=package://g1_description/meshes/dex5_right/right_thumb_4.STL; visual mesh filename=package://g1_description/meshes/dex5_right/right_thumb_4.STL
- added link right_thumb_force_sensor_1, mass 0.000234345870584151; collision mesh filename=package://g1_description/meshes/dex5_right/right_thumb_forc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; visual mesh filename=package://g1_description/meshes/dex5_right/right_thumb_forc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
- added link right_thumb_force_sensor_2, mass 0.000119024197892742; collision mesh filename=package://g1_description/meshes/dex5_right/right_thumb_forc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; visual mesh filename=package://g1_description/meshes/dex5_right/right_thumb_forc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
- added link right_thumb_force_sensor_3, mass 0.000169893832350009; collision mesh filename=package://g1_description/meshes/dex5_right/right_thumb_forc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; visual mesh filename=package://g1_description/meshes/dex5_right/right_thumb_forc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
- added link right_thumb_force_sensor_4, mass 1.66991205082657E-05; collision mesh filename=package://g1_description/meshes/dex5_right/right_thumb_forc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; visual mesh filename=package://g1_description/meshes/dex5_right/right_thumb_forc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
Joints:
- added joint left_dex5_mount_joint: type fixed, parent left_wrist_yaw_link, child left_dex5_base_link, origin xyz=0 0 0 rpy=0 0 0
- added joint left_hand_grasp_frame_joint: type fixed, parent left_plam_1, child left_hand_grasp_frame, origin xyz=0 0 0 rpy=0 0 0
- added joint left_index_1_joint: type revolute, parent left_dex5_base_link, child left_index_1, origin xyz=0.00056467 0.038679 -0.1564 rpy=-1.5359 0 0, axis 0 0 -1, limit lower=0 upper=1.4381 effort=1 velocity=2
- added joint left_index_2_joint: type revolute, parent left_index_1, child left_index_2, origin xyz=0.0034259 0.032596 -0.00055 rpy=0 0 0, axis 0 0 -1, limit lower=0 upper=1.476374 effort=1 velocity=2, mimic joint=left_index_1_joint multiplier=1.0843 offset=0
- added joint left_index_force_sensor_1_joint: type fixed, parent left_index_1, child left_index_force_sensor_1, origin xyz=0.012046 0.019649 -0.006651 rpy=-1.5708 1.5351 -1.3587, axis 0 0 0
- added joint left_index_force_sensor_2_joint: type fixed, parent left_index_2, child left_index_force_sensor_2, origin xyz=0.0081655 0.037446 -0.0060795 rpy=-0.037141 0 -0.34877, axis 0 0 0
- added joint left_index_force_sensor_3_joint: type fixed, parent left_index_2, child left_index_force_sensor_3, origin xyz=0.0086237 0.052572 -0.0060954 rpy=-1.5708 1.5252 -0.87237, axis 0 0 0
- added joint left_little_1_joint: type revolute, parent left_dex5_base_link, child left_little_1, origin xyz=0.00056467 -0.025916 -0.15365 rpy=-1.6755 0 0, axis 0 0 -1, limit lower=0 upper=1.4381 effort=1 velocity=2
- added joint left_little_2_joint: type revolute, parent left_little_1, child left_little_2, origin xyz=0.0034259 0.032596 -0.00055 rpy=0 0 0, axis 0 0 -1, limit lower=0 upper=1.476374 effort=1 velocity=2, mimic joint=left_little_1_joint multiplier=1.0843 offset=0
- added joint left_little_force_sensor_1_joint: type fixed, parent left_little_1, child left_little_force_sensor_1, origin xyz=0.012046 0.019649 -0.006651 rpy=1.5708 1.4637 1.7829, axis 0 0 0
- added joint left_little_force_sensor_2_joint: type fixed, parent left_little_2, child left_little_force_sensor_2, origin xyz=0.0064514 0.027683 -0.0061172 rpy=1.5708 1.4597 1.2289, axis 0 0 0
- added joint left_little_force_sensor_3_joint: type fixed, parent left_little_2, child left_little_force_sensor_3, origin xyz=0.0063973 0.042707 -0.0061154 rpy=1.5708 1.4336 2.2761, axis 0 0 0
- added joint left_middle_1_joint: type revolute, parent left_dex5_base_link, child left_middle_1, origin xyz=0.00056467 0.0171 -0.157 rpy=-1.5708 0 0, axis 0 0 -1, limit lower=0 upper=1.4381 effort=1 velocity=2
- added joint left_middle_2_joint: type revolute, parent left_middle_1, child left_middle_2, origin xyz=0.0034259 0.032596 -0.00055 rpy=0 0 0, axis 0 0 -1, limit lower=0 upper=1.476374 effort=1 velocity=2, mimic joint=left_middle_1_joint multiplier=1.0843 offset=0
- added joint left_middle_force_sensor_1_joint: type fixed, parent left_middle_1, child left_middle_force_sensor_1, origin xyz=0.012046 0.019649 -0.006651 rpy=-1.9353 1.5708 -1.7232, axis 0 0 0
- added joint left_middle_force_sensor_2_joint: type fixed, parent left_middle_2, child left_middle_force_sensor_2, origin xyz=0.009086 0.040962 -0.0061003 rpy=-1.0917 1.5708 -1.4646, axis 0 0 0
- added joint left_middle_force_sensor_3_joint: type fixed, parent left_middle_2, child left_middle_force_sensor_3, origin xyz=0.0098294 0.056051 -0.0061006 rpy=-2.1401 1.5708 -1.4657, axis 0 0 0
- added joint left_plam_1_joint: type fixed, parent left_dex5_base_link, child left_plam_1, origin xyz=0 0 -0.031 rpy=-3.1416 0 0, axis 0 0 0
- added joint left_plam_2_joint: type fixed, parent left_plam_1, child left_plam_2, origin xyz=0 0 0 rpy=0 0 0, axis 0 0 0
- added joint left_plam_force_sensor_joint: type fixed, parent left_plam_1, child left_plam_force_sensor, origin xyz=0.012296 -0.00036819 0.088601 rpy=1.5708 0 1.5708, axis 0 0 0
- added joint left_ring_1_joint: type revolute, parent left_dex5_base_link, child left_ring_1, origin xyz=0.00056467 -0.0045302 -0.15683 rpy=-1.6232 0 0, axis 0 0 -1, limit lower=0 upper=1.4381 effort=1 velocity=2
- added joint left_ring_2_joint: type revolute, parent left_ring_1, child left_ring_2, origin xyz=0.0034259 0.032596 -0.00055 rpy=0 0 0, axis 0 0 -1, limit lower=0 upper=1.476374 effort=1 velocity=2, mimic joint=left_ring_1_joint multiplier=1.0843 offset=0
- added joint left_ring_force_sensor_1_joint: type fixed, parent left_ring_1, child left_ring_force_sensor_1, origin xyz=0.012046 0.019649 -0.006651 rpy=1.5708 1.5172 1.7829, axis 0 0 0
- added joint left_ring_force_sensor_2_joint: type fixed, parent left_ring_2, child left_ring_force_sensor_2, origin xyz=0.0081655 0.037446 -0.0060795 rpy=1.5708 1.5151 1.222, axis 0 0 0
- added joint left_ring_force_sensor_3_joint: type fixed, parent left_ring_2, child left_ring_force_sensor_3, origin xyz=0.0086237 0.052572 -0.0060954 rpy=1.5708 1.5025 2.2692, axis 0 0 0
- added joint left_thumb_1_joint: type revolute, parent left_dex5_base_link, child left_thumb_1, origin xyz=0.02101 0.0269 -0.0826 rpy=3.1416 0 0, axis 0 0 1, limit lower=0 upper=1.658 effort=1 velocity=2
- added joint left_thumb_2_joint: type revolute, parent left_thumb_1, child left_thumb_2, origin xyz=0.013438 -0.012862 -0.0076 rpy=1.5708 0 -1.5708, axis 0.17365 0 0.98481, limit lower=0 upper=0.62 effort=1 velocity=2
- added joint left_thumb_3_joint: type revolute, parent left_thumb_2, child left_thumb_3, origin xyz=0.052954 0.032799 -0.0093372 rpy=0 0 0, axis 0.17365 0 0.98481, limit lower=0 upper=0.5410520681182421 effort=1 velocity=2, mimic joint=left_thumb_2_joint multiplier=0.8392 offset=0
- added joint left_thumb_4_joint: type revolute, parent left_thumb_3, child left_thumb_4, origin xyz=0.01865 0.013373 -0.0022731 rpy=0 0 0, axis 0.17365 0 0.98481, limit lower=0 upper=0.45553093477052004 effort=1 velocity=2, mimic joint=left_thumb_3_joint multiplier=0.891 offset=0
- added joint left_thumb_force_sensor_1_joint: type fixed, parent left_thumb_2, child left_thumb_force_sensor_1, origin xyz=0.023412 0.033251 0.0070079 rpy=1.1285 1.3976 3.1383, axis 0 0 0
- added joint left_thumb_force_sensor_2_joint: type fixed, parent left_thumb_3, child left_thumb_force_sensor_2, origin xyz=0.0080283 0.016443 0.00982 rpy=0.96258 1.4071 3.0993, axis 0 0 0
- added joint left_thumb_force_sensor_3_joint: type fixed, parent left_thumb_4, child left_thumb_force_sensor_3, origin xyz=0.0076349 0.020486 0.0088094 rpy=0.64092 1.3963 -3.1415, axis 0 0 0
- added joint left_thumb_force_sensor_4_joint: type fixed, parent left_thumb_4, child left_thumb_force_sensor_4, origin xyz=0.018831 0.027914 0.0068352 rpy=1.7521 1.3962 -3.1401, axis 0 0 0
- added joint right_dex5_mount_joint: type fixed, parent right_wrist_yaw_link, child right_dex5_base_link, origin xyz=0 0 0 rpy=0 0 0
- added joint right_hand_grasp_frame_joint: type fixed, parent right_plam_1, child right_hand_grasp_frame, origin xyz=0 0 0 rpy=0 0 0
- added joint right_index_1_joint: type revolute, parent right_dex5_base_link, child right_index_1, origin xyz=0.00056467 -0.038679 -0.1564 rpy=-1.6057 0 0, axis 0 0 -1, limit lower=0 upper=1.4381 effort=1 velocity=1
- added joint right_index_2_joint: type revolute, parent right_index_1, child right_index_2, origin xyz=0.0034259 0.032596 0.00055 rpy=0 0 0, axis 0 0 -1, limit lower=0 upper=1.476374 effort=1 velocity=1, mimic joint=right_index_1_joint multiplier=1.0843 offset=0
- added joint right_index_force_sensor_1_joint: type fixed, parent right_index_1, child right_index_force_sensor_1, origin xyz=0.012046 0.019649 0.006651 rpy=1.5708 1.5351 1.7829, axis 0 0 0
- added joint right_index_force_sensor_2_joint: type fixed, parent right_index_2, child right_index_force_sensor_2, origin xyz=0.0081655 0.037446 0.0060795 rpy=1.5708 1.5337 1.222, axis 0 0 0
- added joint right_index_force_sensor_3_joint: type fixed, parent right_index_2, child right_index_force_sensor_3, origin xyz=0.0086237 0.052572 0.0060954 rpy=1.5708 1.5252 2.2692, axis 0 0 0
- added joint right_little_1_joint: type revolute, parent right_dex5_base_link, child right_little_1, origin xyz=0.00056467 0.025916 -0.15365 rpy=-1.4661 0 0, axis 0 0 -1, limit lower=0 upper=1.4381 effort=1 velocity=1
- added joint right_little_2_joint: type revolute, parent right_little_1, child right_little_2, origin xyz=0.0034259 0.032596 0.00055 rpy=0 0 0, axis 0 0 -1, limit lower=0 upper=1.476374 effort=1 velocity=1, mimic joint=right_little_1_joint multiplier=1.0843 offset=0
- added joint right_little_force_sensor_1_joint: type fixed, parent right_little_1, child right_little_force_sensor_1, origin xyz=0.012046 0.019649 0.006651 rpy=-1.5708 1.4637 -1.3587, axis 0 0 0
- added joint right_little_force_sensor_2_joint: type fixed, parent right_little_2, child right_little_force_sensor_2, origin xyz=0.0064512 0.027683 0.0061172 rpy=-1.5708 1.4597 -1.9127, axis 0 0 0
- added joint right_little_force_sensor_3_joint: type fixed, parent right_little_2, child right_little_force_sensor_3, origin xyz=0.0063972 0.042707 0.0061154 rpy=-1.5708 1.4336 -0.86551, axis 0 0 0
- added joint right_middle_1_joint: type revolute, parent right_dex5_base_link, child right_middle_1, origin xyz=0.00056467 -0.0171 -0.157 rpy=-1.5708 0 0, axis 0 0 -1, limit lower=0 upper=1.4381 effort=1 velocity=1
- added joint right_middle_2_joint: type revolute, parent right_middle_1, child right_middle_2, origin xyz=0.0034259 0.032596 0.00055 rpy=0 0 0, axis 0 0 -1, limit lower=0 upper=1.476374 effort=1 velocity=1, mimic joint=right_middle_1_joint multiplier=1.0843 offset=0
- added joint right_middle_force_sensor_1_joint: type fixed, parent right_middle_1, child right_middle_force_sensor_1, origin xyz=0.012046 0.019649 0.006651 rpy=-0.21209 1.5708 0, axis 0 0 0
- added joint right_middle_force_sensor_2_joint: type fixed, parent right_middle_2, child right_middle_force_sensor_2, origin xyz=0.0090859 0.040963 0.0061003 rpy=0.37285 1.5708 0, axis 0 0 0
- added joint right_middle_force_sensor_3_joint: type fixed, parent right_middle_2, child right_middle_force_sensor_3, origin xyz=0.0098294 0.056051 0.0061006 rpy=-0.67435 1.5708 0, axis 0 0 0
- added joint right_plam_1_joint: type fixed, parent right_dex5_base_link, child right_plam_1, origin xyz=0 0 -0.0305 rpy=3.1416 0 0, axis 0 0 0
- added joint right_plam_2_joint: type fixed, parent right_plam_1, child right_plam_2, origin xyz=0 0 0 rpy=0 0 0, axis 0 0 0
- added joint right_plam_force_sensor_joint: type fixed, parent right_plam_1, child right_plam_force_sensor, origin xyz=0.012296 0.00036819 0.089101 rpy=1.5708 0 1.5708, axis 0 0 0
- added joint right_ring_1_joint: type revolute, parent right_dex5_base_link, child right_ring_1, origin xyz=0.00056467 0.0045302 -0.15683 rpy=-1.5184 0 0, axis 0 0 -1, limit lower=0 upper=1.4381 effort=1 velocity=1
- added joint right_ring_2_joint: type revolute, parent right_ring_1, child right_ring_2, origin xyz=0.0034259 0.032596 0.00055 rpy=0 0 0, axis 0 0 -1, limit lower=0 upper=1.476374 effort=1 velocity=1, mimic joint=right_ring_1_joint multiplier=1.0843 offset=0
- added joint right_ring_force_sensor_1_joint: type fixed, parent right_ring_1, child right_ring_force_sensor_1, origin xyz=0.012046 0.019649 0.006651 rpy=-1.5708 1.5172 -1.3587, axis 0 0 0
- added joint right_ring_force_sensor_2_joint: type fixed, parent right_ring_2, child right_ring_force_sensor_2, origin xyz=0.0081655 0.037446 0.0060795 rpy=-1.5708 1.5151 -1.9196, axis 0 0 0
- added joint right_ring_force_sensor_3_joint: type fixed, parent right_ring_2, child right_ring_force_sensor_3, origin xyz=0.0086237 0.052572 0.0060954 rpy=-1.5708 1.5025 -0.87237, axis 0 0 0
- added joint right_thumb_1_joint: type revolute, parent right_dex5_base_link, child right_thumb_1, origin xyz=0.02101 -0.0269 -0.0826 rpy=-3.1416 0 0, axis 0 0 -1, limit lower=0 upper=1.658 effort=1 velocity=2
- added joint right_thumb_2_joint: type revolute, parent right_thumb_1, child right_thumb_2, origin xyz=0.013438 0.012862 -0.0076 rpy=1.5708 0 -1.5708, axis 0.17365 0 -0.98481, limit lower=0 upper=0.62 effort=1 velocity=2
- added joint right_thumb_3_joint: type revolute, parent right_thumb_2, child right_thumb_3, origin xyz=-0.052954 0.032799 -0.0093372 rpy=0 0 0, axis 0.17365 0 -0.98481, limit lower=0 upper=0.5410520681182421 effort=1 velocity=2, mimic joint=right_thumb_2_joint multiplier=0.8392 offset=0
- added joint right_thumb_4_joint: type revolute, parent right_thumb_3, child right_thumb_4, origin xyz=-0.01865 0.013373 -0.0022731 rpy=0 0 0, axis 0.17365 0 -0.98481, limit lower=0 upper=0.45553093477052004 effort=1 velocity=2, mimic joint=right_thumb_3_joint multiplier=0.891 offset=0
- added joint right_thumb_force_sensor_1_joint: type fixed, parent right_thumb_2, child right_thumb_force_sensor_1, origin xyz=-0.023424 0.033251 0.007073 rpy=-0.99905 1.4338 0.13409, axis 0 0 0
- added joint right_thumb_force_sensor_2_joint: type fixed, parent right_thumb_3, child right_thumb_force_sensor_2, origin xyz=-0.0080057 0.016443 0.0096921 rpy=-1.041 1.3851 -0.037357, axis 0 0 0
- added joint right_thumb_force_sensor_3_joint: type fixed, parent right_thumb_4, child right_thumb_force_sensor_3, origin xyz=-0.0076345 0.020486 0.0088067 rpy=-0.64083 1.3963 4.2914E-05, axis 0 0 0
- added joint right_thumb_force_sensor_4_joint: type fixed, parent right_thumb_4, child right_thumb_force_sensor_4, origin xyz=-0.01883 0.027914 0.0068326 rpy=-1.7492 1.3963 0.0014317, axis 0 0 0
