Commit message: Flatten Dex5 models into host URDF
Co-authored-by: Mertsr <115826687+Mertsr@users.noreply.github.com>

File: workspace/src/g1_description/urdf/g1_common.xacro (robot description, xacro)
@@ -1,7 +1,7 @@
 <?xml version="1.0"?>
 <robot xmlns:xacro="http://www.ros.org/wiki/xacro" name="g1_29dof_with_hand_rev_1_0">
-  <!-- The robot without the body's ros2_control block: the vendored body, the frames the stack
-       looks up by name, and both Dex5 hands. Geometry-only consumers (RViz, the sensor-extrinsic
-       test) load this file so they cannot claim the body motors. -->
+  <!-- The plain host URDF contains the G1 body and both Dex5 hands. This file adds shared sensor
+       frames without the body's ros2_control block. Geometry-only consumers (RViz, the
+       sensor-extrinsic test) load it so they cannot claim the body motors. -->
   <!-- Unitree's URDF, byte-for-byte (CRLF included) apart from mesh paths rewritten to
        package:// for RViz. Additions go in this file, so it stays diffable against upstream. -->
@@ -102,39 +102,3 @@
     <origin xyz="0.011 0.02329 -0.04412" rpy="0 0 0"/>
   </joint>
-  <!-- Inspire RH56E2 ("Dex5") hands, SolidWorks exports transcribed as supplied: each file's root
-       is left_dex5_base_link / right_dex5_base_link and its joints are mounted below. Only the
-       mesh URIs differ from the export: package://g1_description/meshes/dex5_left/<name>.STL and
-       .../dex5_right/<name>.STL. The STL files are NOT in the repo; install them at
-       workspace/src/g1_description/meshes/dex5_left/ and .../dex5_right/ (see README).
-       No ros2_control is declared for the hands in this change. -->
-  <xacro:include filename="RH56E2_L_2025_9_10.xacro"/>
-  <xacro:include filename="RH56E2_R_2025_9_11.xacro"/>
-  <!-- PROVISIONAL mount of each hand root on the wrist: zeros, NOT a physically validated fit.
-       Override at xacro time, e.g. xacro g1_lowcmd.urdf.xacro dex5_left_mount_xyz:="0.05 0 0". -->
-  <xacro:arg name="dex5_left_mount_xyz" default="0 0 0"/>
-  <xacro:arg name="dex5_left_mount_rpy" default="0 0 0"/>
-  <xacro:arg name="dex5_right_mount_xyz" default="0 0 0"/>
-  <xacro:arg name="dex5_right_mount_rpy" default="0 0 0"/>
-  <joint name="left_dex5_mount_joint" type="fixed">
-    <parent link="left_wrist_yaw_link"/>
-    <child link="left_dex5_base_link"/>
-    <origin xyz="$(arg dex5_left_mount_xyz)" rpy="$(arg dex5_left_mount_rpy)"/>
-  </joint>
-  <joint name="right_dex5_mount_joint" type="fixed">
-    <parent link="right_wrist_yaw_link"/>
-    <child link="right_dex5_base_link"/>
-    <origin xyz="$(arg dex5_right_mount_xyz)" rpy="$(arg dex5_right_mount_rpy)"/>
-  </joint>
-  <!-- Grasp frames keep their names for consumers, now on the Dex5 roots. PROVISIONAL zero
-       offset: the old Dex3 closing-point offsets do not apply to this hand. -->
-  <xacro:macro name="g1_grasp_frame" params="side mirror">
-    <link name="${side}_hand_grasp_frame"/>
-    <joint name="${side}_hand_grasp_frame_joint" type="fixed">
-      <parent link="${side}_dex5_base_link"/>
-      <child link="${side}_hand_grasp_frame"/>
-      <origin xyz="0 0 0" rpy="0 0 0"/>
-    </joint>
-  </xacro:macro>
-  <xacro:g1_grasp_frame side="left" mirror="-1"/>
-  <xacro:g1_grasp_frame side="right" mirror="1"/>
 </robot>

File: workspace/src/g1_description/urdf/g1_lowcmd.urdf.xacro (robot description, xacro)
@@ -2,5 +2,5 @@
 <robot xmlns:xacro="http://www.ros.org/wiki/xacro" name="g1_29dof_with_hand_rev_1_0">
   <!-- All 29 body motors on G1LowCmdSystem over rt/lowcmd, with no onboard balance underneath.
-       Everything else, including both Dex5 hands (no hand ros2_control yet), comes from g1_common.xacro. -->
+       g1_common.xacro includes the host URDF and adds shared sensor frames. -->
   <xacro:include filename="g1_common.xacro"/>
   <xacro:property name="lowcmd" value="${xacro.load_yaml('../config/lowcmd_params.yaml')}"/>
