Commit message: Replace contents with g1-dex5-mujoco snapshot (1767ca5)
Co-Authored-By: Claude Sonnet 5.5 <noreply@anthropic.com>
Claude-Session: https://claude.ai/code/session_0143uuLoCScApeMYUcosqA6K

File: workspace/src/g1_description/urdf/g1_29dof_with_hand_rev_1_0.urdf (robot description, URDF)
Before this commit: robot g1_29dof_with_hand_rev_1_0, 103 links, 102 joints
Links:
- removed link left_dex5_base_link
- removed link left_hand_grasp_frame
- removed link left_index_1
- removed link left_index_2
- removed link left_index_force_sensor_1
- removed link left_index_force_sensor_2
- removed link left_index_force_sensor_3
- removed link left_little_1
- removed link left_little_2
- removed link left_little_force_sensor_1
- removed link left_little_force_sensor_2
- removed link left_little_force_sensor_3
- removed link left_middle_1
- removed link left_middle_2
- removed link left_middle_force_sensor_1
- removed link left_middle_force_sensor_2
- removed link left_middle_force_sensor_3
- removed link left_plam_1
- removed link left_plam_2
- removed link left_plam_force_sensor
- removed link left_ring_1
- removed link left_ring_2
- removed link left_ring_force_sensor_1
- removed link left_ring_force_sensor_2
- removed link left_ring_force_sensor_3
- removed link left_thumb_1
- removed link left_thumb_2
- removed link left_thumb_3
- removed link left_thumb_4
- removed link left_thumb_force_sensor_1
- removed link left_thumb_force_sensor_2
- removed link left_thumb_force_sensor_3
- removed link left_thumb_force_sensor_4
- removed link right_dex5_base_link
- removed link right_hand_grasp_frame
- removed link right_index_1
- removed link right_index_2
- removed link right_index_force_sensor_1
- removed link right_index_force_sensor_2
- removed link right_index_force_sensor_3
- removed link right_little_1
- removed link right_little_2
- removed link right_little_force_sensor_1
- removed link right_little_force_sensor_2
- removed link right_little_force_sensor_3
- removed link right_middle_1
- removed link right_middle_2
- removed link right_middle_force_sensor_1
- removed link right_middle_force_sensor_2
- removed link right_middle_force_sensor_3
- removed link right_plam_1
- removed link right_plam_2
- removed link right_plam_force_sensor
- removed link right_ring_1
- removed link right_ring_2
- removed link right_ring_force_sensor_1
- removed link right_ring_force_sensor_2
- removed link right_ring_force_sensor_3
- removed link right_thumb_1
- removed link right_thumb_2
- removed link right_thumb_3
- removed link right_thumb_4
- removed link right_thumb_force_sensor_1
- removed link right_thumb_force_sensor_2
- removed link right_thumb_force_sensor_3
- removed link right_thumb_force_sensor_4
- added link left_hand_index_0_link, mass 0.05885070; collision mesh filename=package://g1_description/meshes/left_hand_index_0_link.STL; visual mesh filename=package://g1_description/meshes/left_hand_index_0_link.STL
- added link left_hand_index_1_link, mass 0.02030626; collision mesh filename=package://g1_description/meshes/left_hand_index_1_link.STL; visual mesh filename=package://g1_description/meshes/left_hand_index_1_link.STL
- added link left_hand_middle_0_link, mass 0.05885070; collision mesh filename=package://g1_description/meshes/left_hand_middle_0_link.STL; visual mesh filename=package://g1_description/meshes/left_hand_middle_0_link.STL
- added link left_hand_middle_1_link, mass 0.02030626; collision mesh filename=package://g1_description/meshes/left_hand_middle_1_link.STL; visual mesh filename=package://g1_description/meshes/left_hand_middle_1_link.STL
- added link left_hand_palm_link, mass 0.37283854; collision mesh filename=package://g1_description/meshes/left_hand_palm_link.STL; visual mesh filename=package://g1_description/meshes/left_hand_palm_link.STL
- added link left_hand_thumb_0_link, mass 0.08623657; collision mesh filename=package://g1_description/meshes/left_hand_thumb_0_link.STL; visual mesh filename=package://g1_description/meshes/left_hand_thumb_0_link.STL
- added link left_hand_thumb_1_link, mass 0.05885070; collision box size=0.02 0.03 0.02; visual mesh filename=package://g1_description/meshes/left_hand_thumb_1_link.STL
- added link left_hand_thumb_2_link, mass 0.02030626; collision mesh filename=package://g1_description/meshes/left_hand_thumb_2_link.STL; visual mesh filename=package://g1_description/meshes/left_hand_thumb_2_link.STL
- added link right_hand_index_0_link, mass 0.05885070; collision mesh filename=package://g1_description/meshes/right_hand_index_0_link.STL; visual mesh filename=package://g1_description/meshes/right_hand_index_0_link.STL
- added link right_hand_index_1_link, mass 0.02030626; collision mesh filename=package://g1_description/meshes/right_hand_index_1_link.STL; visual mesh filename=package://g1_description/meshes/right_hand_index_1_link.STL
- added link right_hand_middle_0_link, mass 0.05885070; collision mesh filename=package://g1_description/meshes/right_hand_middle_0_link.STL; visual mesh filename=package://g1_description/meshes/right_hand_middle_0_link.STL
- added link right_hand_middle_1_link, mass 0.02030626; collision mesh filename=package://g1_description/meshes/right_hand_middle_1_link.STL; visual mesh filename=package://g1_description/meshes/right_hand_middle_1_link.STL
- added link right_hand_palm_link, mass 0.37283854; collision mesh filename=package://g1_description/meshes/right_hand_palm_link.STL; visual mesh filename=package://g1_description/meshes/right_hand_palm_link.STL
- added link right_hand_thumb_0_link, mass 0.08623657; collision mesh filename=package://g1_description/meshes/right_hand_thumb_0_link.STL; visual mesh filename=package://g1_description/meshes/right_hand_thumb_0_link.STL
- added link right_hand_thumb_1_link, mass 0.05885070; collision box size=0.02 0.03 0.02; visual mesh filename=package://g1_description/meshes/right_hand_thumb_1_link.STL
- added link right_hand_thumb_2_link, mass 0.02030626; collision mesh filename=package://g1_description/meshes/right_hand_thumb_2_link.STL; visual mesh filename=package://g1_description/meshes/right_hand_thumb_2_link.STL
Joints:
- removed joint left_dex5_mount_joint
- removed joint left_hand_grasp_frame_joint
- removed joint left_index_1_joint
- removed joint left_index_2_joint
- removed joint left_index_force_sensor_1_joint
- removed joint left_index_force_sensor_2_joint
- removed joint left_index_force_sensor_3_joint
- removed joint left_little_1_joint
- removed joint left_little_2_joint
- removed joint left_little_force_sensor_1_joint
- removed joint left_little_force_sensor_2_joint
- removed joint left_little_force_sensor_3_joint
- removed joint left_middle_1_joint
- removed joint left_middle_2_joint
- removed joint left_middle_force_sensor_1_joint
- removed joint left_middle_force_sensor_2_joint
- removed joint left_middle_force_sensor_3_joint
- removed joint left_plam_1_joint
- removed joint left_plam_2_joint
- removed joint left_plam_force_sensor_joint
- removed joint left_ring_1_joint
- removed joint left_ring_2_joint
- removed joint left_ring_force_sensor_1_joint
- removed joint left_ring_force_sensor_2_joint
- removed joint left_ring_force_sensor_3_joint
- removed joint left_thumb_1_joint
- removed joint left_thumb_2_joint
- removed joint left_thumb_3_joint
- removed joint left_thumb_4_joint
- removed joint left_thumb_force_sensor_1_joint
- removed joint left_thumb_force_sensor_2_joint
- removed joint left_thumb_force_sensor_3_joint
- removed joint left_thumb_force_sensor_4_joint
- removed joint right_dex5_mount_joint
- removed joint right_hand_grasp_frame_joint
- removed joint right_index_1_joint
- removed joint right_index_2_joint
- removed joint right_index_force_sensor_1_joint
- removed joint right_index_force_sensor_2_joint
- removed joint right_index_force_sensor_3_joint
- removed joint right_little_1_joint
- removed joint right_little_2_joint
- removed joint right_little_force_sensor_1_joint
- removed joint right_little_force_sensor_2_joint
- removed joint right_little_force_sensor_3_joint
- removed joint right_middle_1_joint
- removed joint right_middle_2_joint
- removed joint right_middle_force_sensor_1_joint
- removed joint right_middle_force_sensor_2_joint
- removed joint right_middle_force_sensor_3_joint
- removed joint right_plam_1_joint
- removed joint right_plam_2_joint
- removed joint right_plam_force_sensor_joint
- removed joint right_ring_1_joint
- removed joint right_ring_2_joint
- removed joint right_ring_force_sensor_1_joint
- removed joint right_ring_force_sensor_2_joint
- removed joint right_ring_force_sensor_3_joint
- removed joint right_thumb_1_joint
- removed joint right_thumb_2_joint
- removed joint right_thumb_3_joint
- removed joint right_thumb_4_joint
- removed joint right_thumb_force_sensor_1_joint
- removed joint right_thumb_force_sensor_2_joint
- removed joint right_thumb_force_sensor_3_joint
- removed joint right_thumb_force_sensor_4_joint
- added joint left_hand_index_0_joint: type revolute, parent left_hand_palm_link, child left_hand_index_0_link, origin xyz=0.0777 0.0016 0.0285 rpy=0 0 0, axis 0 0 1, limit lower=-1.57079632 upper=0 effort=1.4 velocity=12
- added joint left_hand_index_1_joint: type revolute, parent left_hand_index_0_link, child left_hand_index_1_link, origin xyz=0.0458 0 0 rpy=0 0 0, axis 0 0 1, limit lower=-1.74532925 upper=0 effort=1.4 velocity=12
- added joint left_hand_middle_0_joint: type revolute, parent left_hand_palm_link, child left_hand_middle_0_link, origin xyz=0.0777 0.0016 -0.0285 rpy=0 0 0, axis 0 0 1, limit lower=-1.57079632 upper=0 effort=1.4 velocity=12
- added joint left_hand_middle_1_joint: type revolute, parent left_hand_middle_0_link, child left_hand_middle_1_link, origin xyz=0.0458 0 0 rpy=0 0 0, axis 0 0 1, limit lower=-1.74532925 upper=0 effort=1.4 velocity=12
- added joint left_hand_palm_joint: type fixed, parent left_wrist_yaw_link, child left_hand_palm_link, origin xyz=0.0415 0.003 0 rpy=0 0 0
- added joint left_hand_thumb_0_joint: type revolute, parent left_hand_palm_link, child left_hand_thumb_0_link, origin xyz=0.0255 0 0 rpy=0 0 0, axis 0 1 0, limit lower=-1.04719755 upper=1.04719755 effort=2.45 velocity=3.14
- added joint left_hand_thumb_1_joint: type revolute, parent left_hand_thumb_0_link, child left_hand_thumb_1_link, origin xyz=-0.0025 -0.0193 0 rpy=0 0 0, axis 0 0 1, limit lower=-0.61086523 upper=1.04719755 effort=1.4 velocity=12
- added joint left_hand_thumb_2_joint: type revolute, parent left_hand_thumb_1_link, child left_hand_thumb_2_link, origin xyz=0 -0.0458 0 rpy=0 0 0, axis 0 0 1, limit lower=0 upper=1.74532925 effort=1.4 velocity=12
- added joint right_hand_index_0_joint: type revolute, parent right_hand_palm_link, child right_hand_index_0_link, origin xyz=0.0777 -0.0016 0.0285 rpy=0 0 0, axis 0 0 1, limit lower=0 upper=1.57079632 effort=1.4 velocity=12
- added joint right_hand_index_1_joint: type revolute, parent right_hand_index_0_link, child right_hand_index_1_link, origin xyz=0.0458 0 0 rpy=0 0 0, axis 0 0 1, limit lower=0 upper=1.74532925 effort=1.4 velocity=12
- added joint right_hand_middle_0_joint: type revolute, parent right_hand_palm_link, child right_hand_middle_0_link, origin xyz=0.0777 -0.0016 -0.0285 rpy=0 0 0, axis 0 0 1, limit lower=0 upper=1.57079632 effort=1.4 velocity=12
- added joint right_hand_middle_1_joint: type revolute, parent right_hand_middle_0_link, child right_hand_middle_1_link, origin xyz=0.0458 0 0 rpy=0 0 0, axis 0 0 1, limit lower=0 upper=1.74532925 effort=1.4 velocity=12
- added joint right_hand_palm_joint: type fixed, parent right_wrist_yaw_link, child right_hand_palm_link, origin xyz=0.0415 -0.003 0 rpy=0 0 0
- added joint right_hand_thumb_0_joint: type revolute, parent right_hand_palm_link, child right_hand_thumb_0_link, origin xyz=0.0255 0 0 rpy=0 0 0, axis 0 1 0, limit lower=-1.04719755 upper=1.04719755 effort=2.45 velocity=3.14
- added joint right_hand_thumb_1_joint: type revolute, parent right_hand_thumb_0_link, child right_hand_thumb_1_link, origin xyz=-0.0025 0.0193 0 rpy=0 0 0, axis 0 0 1, limit lower=-1.04719755 upper=0.61086523 effort=1.4 velocity=12
- added joint right_hand_thumb_2_joint: type revolute, parent right_hand_thumb_1_link, child right_hand_thumb_2_link, origin xyz=0 0.0458 0 rpy=0 0 0, axis 0 0 1, limit lower=-1.74532925 upper=0 effort=1.4 velocity=12
